Commit message: Optatert vinkel på robot

File: src/my_robot_cell_description/urdf/my_robot_cell_macro.xacro (robot description, xacro)
@@ -121,5 +121,5 @@
       physical_parameters_file="${physical_parameters_file}"
       visual_parameters_file="${visual_parameters_file}">
-      <origin xyz="0.575 0.365 0.015" rpy="0 0 0"/>
+      <origin xyz="0.575 0.365 0.015" rpy="0 0 -0.7854"/>
     </xacro:ur_robot>
     <!-- Robot 2 -->
@@ -132,5 +132,5 @@
       physical_parameters_file="${physical_parameters_file}"
       visual_parameters_file="${visual_parameters_file}">
-      <origin xyz="-0.425 0.365 0.015" rpy="0 0 0"/>
+      <origin xyz="-0.425 0.365 0.015" rpy="0 0 0.7854"/>
     </xacro:ur_robot>
   </xacro:macro>

Commit message: working

File: src/my_robot_cell_description/urdf/my_robot_cell_macro.xacro (robot description, xacro)
@@ -53,5 +53,5 @@
     <!-- Fest camera_mount til tool0 -->
     <joint name="camera_mount_joint" type="fixed">
-      <parent link="tool0"/>
+      <parent link="${ur_type}_tool0"/>
       <child link="camera_mount"/>
       <origin xyz="0 0 0" rpy="0 0 0"/>
@@ -115,5 +115,5 @@
     <xacro:ur_robot
       name="${ur_type}"
-      tf_prefix=""
+      tf_prefix="${ur_type}_"
       parent="robot_mount"
       joint_limits_parameters_file="${joint_limits_parameters_file}"
@@ -125,6 +125,6 @@
     <!-- Robot 2 -->
     <xacro:ur_robot
-      name="${ur_type}"
-      tf_prefix="_2"
+      name="${ur_type}_2"
+      tf_prefix="${ur_type}_2_"
       parent="robot_mount"
       joint_limits_parameters_file="${joint_limits_parameters_file}"

Commit message: Kamera

File: src/my_robot_cell_description/urdf/my_robot_cell_macro.xacro (robot description, xacro)
@@ -19,5 +19,5 @@
       <visual>
         <geometry>
-          <box size="1.25 0.85 1"/>  <!-- bredde, dybde, høyde -->
+          <box size="1.25 0.85 1"/>
         </geometry>
         <origin rpy="0 0 0" xyz="0.77 0.5 -0.5"/>
@@ -33,5 +33,5 @@
       </collision>
     </link>
-        <!-- Camera mount på tool0 -->
+        <!-- Camera mount on tool0 -->
     <link name="camera_mount">
       <visual>
@@ -51,5 +51,5 @@
       </collision>
     </link>
-    <!-- Fest camera_mount til tool0 -->
+    <!-- Fix camera_mount to tool0 -->
     <joint name="camera_mount_joint" type="fixed">
       <parent link="${ur_type}_tool0"/>
@@ -102,5 +102,5 @@
   </collision>
 </link>
-<!-- Fest til bordet -->
+<!-- Fix to table -->
 <joint name="plate1_joint" type="fixed">
   <parent link="table"/>
@@ -111,5 +111,4 @@
   <child link="plate_2"/>
 </joint>
-    <!--This will create the specific robot-->
     <!-- Robot 1 -->
     <xacro:ur_robot

Commit message: new working code

File: src/my_robot_cell_description/urdf/my_robot_cell_macro.xacro (robot description, xacro)
@@ -19,5 +19,5 @@
       <visual>
         <geometry>
-          <box size="1.25 0.85 1"/>  <!-- bredde, dybde, høyde -->
+          <box size="1.25 0.85 1"/>
         </geometry>
         <origin rpy="0 0 0" xyz="0.77 0.5 -0.5"/>
@@ -33,5 +33,5 @@
       </collision>
     </link>
-        <!-- Camera mount på tool0 -->
+        <!-- Camera mount on tool0 -->
     <link name="camera_mount">
       <visual>
@@ -51,5 +51,5 @@
       </collision>
     </link>
-    <!-- Fest camera_mount til tool0 -->
+    <!-- Fix camera_mount to tool0 -->
     <joint name="camera_mount_joint" type="fixed">
       <parent link="${ur_type}_tool0"/>
@@ -102,5 +102,5 @@
   </collision>
 </link>
-<!-- Fest til bordet -->
+<!-- Fix to table -->
 <joint name="plate1_joint" type="fixed">
   <parent link="table"/>
@@ -111,5 +111,4 @@
   <child link="plate_2"/>
 </joint>
-    <!--This will create the specific robot-->
     <!-- Robot 1 -->
     <xacro:ur_robot
@@ -121,5 +120,5 @@
       physical_parameters_file="${physical_parameters_file}"
       visual_parameters_file="${visual_parameters_file}">
-      <origin xyz="0.575 0.365 0.015" rpy="0 0 -0.7854"/>
+      <origin xyz="0.575 0.365 0.015" rpy="0 0 -3.9254"/>
     </xacro:ur_robot>
     <!-- Robot 2 -->
